Commit message: fix minor bug in dt computation

File: thirdparty/summit_xl/summit_xl_common/summit_xl_description/robots/summit_xl.urdf.xacro (robot description, xacro)
@@ -58,5 +58,5 @@
 	</xacro:landing_platform>
 	<xacro:landing_indicator name="landing_indicator" parent="landing_platform" >
-		<origin xyz="0.55 0.0 0.0" rpy="0 0 0"/>
+		<origin xyz="0.6 0.0 0.0" rpy="0 0 0"/>
 	</xacro:landing_indicator>
 	<!-- SENSORS -->

File: thirdparty/summit_xl/summit_xl_common/summit_xl_description/urdf/platform/landing_indicator.urdf.xacro (robot description, xacro)
@@ -2,6 +2,6 @@
 <robot name="landing_indicator" xmlns:xacro="http://www.ros.org/wiki/xacro">
   <!-- indicator -->
-  <xacro:property name="indicator_length_x" value="0.3" />
-  <xacro:property name="indicator_width_y" value="0.8" />
+  <xacro:property name="indicator_length_x" value="0.2" />
+  <xacro:property name="indicator_width_y" value="1.0" />
   <xacro:property name="indicator_height_z" value="0.01" />
   <xacro:property name="indicator_mass" value="0.2" /> <!-- in kg-->

File: thirdparty/summit_xl/summit_xl_common/summit_xl_description/urdf/platform/landing_platform.urdf.xacro (robot description, xacro)
@@ -2,6 +2,6 @@
 <robot name="landing_platform" xmlns:xacro="http://www.ros.org/wiki/xacro">
   <!-- PLATFORM -->
-  <xacro:property name="platform_length_x" value="0.8" />
-  <xacro:property name="platform_width_y" value="0.8" />
+  <xacro:property name="platform_length_x" value="1.0" />
+  <xacro:property name="platform_width_y" value="1.0" />
   <xacro:property name="platform_height_z" value="0.01" />
   <xacro:property name="platform_mass" value="0.5" /> <!-- in kg-->
